File: Hardware/STM32_Industrial_Edge_Gateway_v0.2.0/STM32_Industrial_Edge_Gateway_v0.2.0.kicad_sch (KiCad schematic)
At the start: 25 parts, among them J1 DC Power Jack (5.5 x 2.1mm), Q1 IRLML6402, U1 MP2338GTL-Z, U2 TLV76733DRVx

Commit message: STM32 MCU Core Schematic
Parts:
- added C10: 100pF, symbol Device:C
- added C11, C18: 1uF, symbol Device:C
- added C12, C13, C14, C15, C16, C17, C19: 100nF, symbol Device:C
- added C20, C21: 2.2µF, symbol Device:C
- added C8, C9: 22pF, symbol Device:C
- added J2: Conn_01x02, symbol Connector_Generic:Conn_01x02
- added J3: Conn_01x05, symbol Connector_Generic:Conn_01x05
- added L2: BLM18AG601SN1D, FILTER_BLM18AG_MUR, symbol BLM18AG601SN1D:BLM18AG601SN1D
- added R10, R9: 10k, symbol Device:R
- added SW1: SW_Push, symbol Switch:SW_Push
- added U3: STM32F407VGTx, Package_QFP:LQFP-100_14x14mm_P0.5mm, symbol MCU_ST_STM32F4:STM32F407VGTx
- added Y1: ECS-80-10-33-CHN-TR, ECS-80-10-33-CHN-TR:XTAL_ECS-80-10-33-CHN-TR, symbol ECS-80-10-33-CHN-TR:ECS-80-10-33-CHN-TR
- renumbered C1A1 to CA1, C2A1 to CA2, C1B1 to CB1, C2B1 to CB2
Connections:
- net +3.3V: now also C12.1, C13.1, C14.1, C15.1, C16.1, C17.1, C18.1, C18.2, C19.1, C19.2, J2.1 (Pin_1), J3.5 (Pin_5), L2.1, R10.2, U3.100 (VDD), U3.11 (VDD), U3.19 (VDD), U3.28 (VDD), U3.50 (VDD), U3.6 (VBAT), U3.75 (VDD)
- net +5V: now also C5.1, R2.1; no longer C5.2, R2.2
- net GND: now also C4.2, C10.1, C11.1, C12.2, C13.2, C14.2, C15.2, C16.2, C17.2, C20.2, C21.2, C8.1, C9.1, J3.4 (Pin_4), R9.2, SW1.1, U3.10 (VSS), U3.20 (VSSA), U3.27 (VSS), U3.74 (VSS), U3.99 (VSS), Y1.2 (GND), Y1.4 (GND); no longer C4.1
- net at R3.2, R7.2: now also C5.2, R2.2; no longer C5.1, R2.1
- net PG: now reaches R6.2, U1.1 (PG)
- net at U1.7 (SS): now also C4.1; no longer C4.2
- new net: C21.1, U3.73 (VCAP_2)
- new net: J2.2 (Pin_2), R9.1, U3.94 (BOOT0)
- new net: C20.1, U3.49 (VCAP_1)
- new net NRST: J3.3 (Pin_3), R10.1, SW1.2, U3.14 (NRST)
- new net OSC_IN: C8.2, U3.12 (PH0), Y1.1 (IN/OUT)
- new net OSC_OUT: C9.2, U3.13 (PH1), Y1.3 (OUT/IN)
- new net SWCLK: J3.2 (Pin_2), U3.76 (PA14)
- new net SWDIO: J3.1 (Pin_1), U3.72 (PA13)
- new net VREF+: C10.2, C11.2, L2.2, U3.21 (VREF+), U3.22 (VDDA)
Other:
- note removed: "Power Supply"
- title: STM32 Industrial Edge Gateway -> STM32 Industrial Edge Gateway - v0.2.0
- moved on the sheet: C3, C4, C5, C6, C7, CA1, CA2, CB1, CB2, D1, D2, F1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

Commit message: Complete schematic
Parts:
- removed D1: SMAF14A, symbol Device:D_TVS
- removed Q1: IRLML6402, Package_TO_SOT_SMD:SOT-23, symbol Transistor_FET:IRLML6402
- removed Y1: ECS-80-10-33-CHN-TR, ECS-80-10-33-CHN-TR:XTAL_ECS-80-10-33-CHN-TR, symbol ECS-80-10-33-CHN-TR:ECS-80-10-33-CHN-TR
- added C1, C23, C24, C25, C26: 100nF, symbol Device:C
- added C2, C22: 18pF, symbol Device:C
- added C27: 10uF, symbol Device:C
- added D1: SMAJ15A, Diode_SMD:D_SMA, symbol Diode:SMAJ15A
- added D3: SM712_SOT23, Package_TO_SOT_SMD:SOT-23, symbol Diode:SM712_SOT23
- added D4, D5: WS2812B, LED_SMD:LED_WS2812B_PLCC4_5.0x5.0mm_P3.2mm, symbol LED:WS2812B
- added J4: HR911105A, HR911105A:HANRUN_HR911105A, symbol HR911105A:HR911105A
- added J5: Screw_Terminal_01x02, symbol Connector:Screw_Terminal_01x02
- added J6: Micro_SD_Card_Det_Hirose_DM3AT, symbol Connector:Micro_SD_Card_Det_Hirose_DM3AT
- added L3, L4: BLM18AG601SN1D, FILTER_BLM18AG_MUR, symbol BLM18AG601SN1D:BLM18AG601SN1D
- added Q2: AO3407A, AO3407A:SOT95P280X125-3N, symbol AO3407A:AO3407A
- added R11, R12: 330, symbol Device:R
- added R13: 120, symbol Device:R
- added R14, R15: 680, symbol Device:R
- added R16, R17, R18, R19: 10k, symbol Device:R
- added R20: 12.1k, symbol Device:R
- added U4: SMD3225, SMD3225:SMD3225, symbol SMD3225:SMD3225
- added U5: LAN8742A, Package_DFN_QFN:VQFN-24-1EP_4x4mm_P0.5mm_EP2.5x2.5mm_ThermalVias, symbol Interface_Ethernet:LAN8742A
- added U6: SRV05-4, Package_TO_SOT_SMD:SOT-23-6, symbol Power_Protection:SRV05-4
- added U7: MAX3485, Package_SO:SOIC-8_3.9x4.9mm_P1.27mm, symbol Interface_UART:MAX3485
- added Y1: ABM8G-25.000MHZ-B4Y-T3, ABM8G-25.000MHZ-B4Y-T3:XTAL_ABM8G-25.000MHZ-B4Y-T3, symbol ABM8G-25.000MHZ-B4Y-T3:ABM8G-25.000MHZ-B4Y-T3
- F1: value Fuse -> 2A Fuse
- J1: value DC Power Jack (5.5 x 2.1mm) -> DC Barrel Jack (5.5 × 2.1mm)
- R8: value 150 -> 330
Connections:
- net +12V: now also Q2.3
- net +3.3V: now also C1.1, C25.2, C26.1, C27.1, J4.12, J4.9, J6.4 (VDD), L3.1, L4.1, R14.1, R15.2, R16.2, R17.2, R18.2, R19.2, U6.5 (VP), U7.8 (VCC)
- net +5V: now also D4.1 (VDD), D5.1 (VDD)
- net GND: now also U3.82 (PD1), C2.2, C22.2, C23.2, C24.2, C25.1, C26.2, C27.2, D1.2 (A2), D3.3 (common), D4.3 (VSS), D5.3 (VSS), J4.15 (SHIELD), J4.16 (SHIELD), J4.8, J6.10 (DET_A), J6.6 (VSS), J6.9 (DET_B), J6.SH (SHIELD), R16.1, R20.1, U4.2, U4.4, U6.2 (VN), U7.5 (GND), Y1.2 (GND), Y1.4 (GND)
- net NRST: now also U5.15 (~{RST})
- net OSC_IN: now also U4.1
- net OSC_OUT: now also U4.3
- net at R1.2: now also Q2.1
- net at F1.2: now also D1.1 (A1), Q2.2
- net MDC: now reaches U3.16 (PC1)
- net MDC: now also U5.13 (MDC)
- net REF_CLK: now reaches U3.24 (PA1)
- net REF_CLK: now also U5.14 (~{INT}/REFCLKO)
- net MDIO: now reaches U3.25 (PA2)
- net MDIO: now also U5.12 (MDIO)
- net SPI1_SCK: now reaches U3.30 (PA5)
- net SPI1_SCK: now also J6.5 (CLK)
- net SPI1_MISO: now reaches U3.31 (PA6)
- net SPI1_MISO: now also J6.7 (DAT0), R19.1
- net CRS_DV: now reaches U3.32 (PA7)
- net CRS_DV: now also U5.11 (CRS_DV/MODE2)
- net RXD0: now reaches U3.33 (PC4)
- net RXD0: now also U5.8 (RXD0/MODE0)
- net RXD1: now reaches U3.34 (PC5)
- net RXD1: now also U5.7 (RXD1/MODE1)
- net TX_EN: now reaches U3.48 (PB11)
- net TX_EN: now also U5.16 (TXEN)
- net TXD0: now reaches U3.51 (PB12)
- net TXD0: now also U5.17 (TXD0)
- net TXD1: now reaches U3.52 (PB13)
- net TXD1: now also U5.18 (TXD1)
- net USART1_TX: now reaches U3.68 (PA9)
- net USART1_TX: now also U7.4 (DI)
- net USART1_RX: now reaches U3.69 (PA10)
- net USART1_RX: now also U7.1 (RO)
- net GPIO_MAX3485: now reaches U3.70 (PA11)
- net GPIO_MAX3485: now also U7.2 (~{RE}), U7.3 (DE)
- net LED_MODBUS: now reaches U3.71 (PA12)
- net LED_MODBUS: now also D4.4 (DIN)
- net SD_CARD_CS: now reaches U3.81 (PD0)
- net SD_CARD_CS: now also J6.2 (DAT3/CD), R17.1
- net LED_SD_CARD: now reaches U3.83 (PD2)
- net LED_SD_CARD: now also D5.4 (DIN)
- net SPI1_MOSI: now reaches U3.91 (PB5)
- net SPI1_MOSI: now also J6.3 (CMD), R18.1
- new net: C24.1, J4.4, L4.2
- new net: R20.2, U5.24 (RBIAS)
- new net: D3.1 (A1), J5.1 (Pin_1), R13.1, R14.2, U7.6 (A)
- new net: D3.2 (A2), J5.2 (Pin_2), R13.2, R15.1, U7.7 (B)
- new net: C23.1, J4.5, L3.2
- new net: C1.2, U5.9 (VDDIO)
- new net: R11.1, U5.2 (LED2/~{INTSEL})
- new net: J4.11, R11.2
- new net: J4.10, R12.2
- new net: C2.1, U5.5 (XTAL1/CLKIN), Y1.1
- new net: C22.1, U5.4 (XTAL2), Y1.3
- new net: R12.1, U5.3 (LED1/REGOFF)
- new net IO1: J4.1
- new net IO2: J4.2
- new net IO3: J4.3
- new net IO4: J4.6
- new net RXN: U5.22 (RXN), U6.6 (IO4)
- new net RXP: U5.23 (RXP), U6.4 (IO3)
- new net TXN: U5.20 (TXN), U6.3 (IO2)
- new net TXP: U5.21 (TXP), U6.1 (IO1)
Other:
- moved on the sheet: C10, C11, C12, C13, C14, C15, C16, C17, C18, C19, C20, C21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

Commit message: Update Ethernet Interface schematic
Connections:
- net GND: now also U5.25 (VSS)
Changed lines of the file:
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@@
 	(wire
 		(pts
+			(xy 63.5 193.04) (xy 66.04 193.04)
+		)
+		(stroke
+			(width 0)
+			(type default)
+		)
+	)
+	(wire
+		(pts
 			(xy 77.47 121.92) (xy 78.74 121.92)
 		)
@@
 	(wire
 		(pts
-			(xy 63.5 193.04) (xy 66.04 193.04)
-		)
-		(stroke
-			(width 0)
-			(type default)
-		)
-	)
-	(wire
-		(pts
 			(xy 45.72 215.9) (xy 50.8 215.9)
 		)
@@
 					(unit 1)
 				)
+			)
+		)
+	)
+	(symbol
+		(lib_id "power:GND")
+		(at 71.12 251.46 0)
+		(unit 1)
+		(body_style 1)
+		(exclude_from_sim no)
+		(in_bom yes)
+		(on_board yes)
+		(in_pos_files yes)
+		(dnp no)
+		(fields_autoplaced yes)
+		(property "Reference" "#PWR067"
+			(at 71.12 257.81 0)
+			(hide yes)
+			(show_name no)
+			(do_not_autoplace no)
+			(effects
+				(font
+					(size 1.27 1.27)
+				)
+			)
+		)
+		(property "Value" "GND"
+			(at 71.12 256.54 0)
+			(show_name no)
+			(do_not_autoplace no)
+			(effects
+				(font
+					(size 1.27 1.27)
+				)
+			)
+		)
+		(property "Footprint" ""
+			(at 71.12 251.46 0)
+			(hide yes)
+			(show_name no)
+			(do_not_autoplace no)
+			(effects
+				(font
+					(size 1.27 1.27)
+				)
+			)
+		)
+		(property "Datasheet" ""
+			(at 71.12 251.46 0)
+			(hide yes)
+			(show_name no)
+			(do_not_autoplace no)
+			(effects
+				(font
+					(size 1.27 1.27)
+				)
+			)
+		)
+		(property "Description" "Power symbol creates a global label with name \"GND\" , ground"
+			(at 71.12 251.46 0)
+			(hide yes)
+			(show_name no)
+			(do_not_autoplace no)
+			(effects
+				(font
+					(size 1.27 1.27)
+				)
+			)
+		)
+		(pin "1"
+		)
+		(instances
+			(project "STM32_Industrial_Edge_Gateway_v0.2.0"
+				(path "/abc15c43-296c-4c96-9fe3-be02bbc91336"
+					(reference "#PWR067")
+					(unit 1)
+				)
